Commit message: Switch mj_kdl backend to ACHD→RNEA two-step torque pipeline
Replace getTotalTorque() with an explicit RNEA pass so qfrc_applied
receives M*qdd + C*qd + G rather than the ACHD internal accumulator.
Add init_env / on_reset / time-backwards reset handling. Fix gravity
sign for RNEA (negate root_acc). Regenerate all existing outputs.

File: thirdparty/kinova/GEN3_URDF_V12.urdf (robot description, URDF)
Before this commit: robot GEN3_URDF_V12, 9 links, 8 joints
Links:
- link Bracelet_Link: mass 0.5006 -> 0.95006
