Commit message: support real Kinova control with ft and gripper

File: thirdparty/kinova/GEN3_URDF_V12.urdf (robot description, URDF)
Before this commit: robot GEN3_URDF_V12, 9 links, 8 joints
Links:
- removed link Bracelet_Link
- removed link EndEffector_Link
- removed link ForeArm_Link
- removed link HalfArm1_Link
- removed link HalfArm2_Link
- removed link Shoulder_Link
- removed link SphericalWrist1_Link
- removed link SphericalWrist2_Link
- added link bracelet_link, mass 0.95006; collision mesh filename=package://kortex_description/arms/gen3/meshes/Bracelet_Link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; visual mesh filename=package://kortex_description/arms/gen3/meshes/Bracelet_Link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
- added link end_effector_link, mass 1.195
- added link forearm_link, mass 0.9302; collision mesh filename=package://kortex_description/arms/gen3/meshes/ForeArm_Link.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; visual mesh filename=package://kortex_description/arms/gen3/meshes/ForeArm_Link.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
- added link ft_sensor_link
- added link half_arm_1_link, mass 1.1636; collision mesh filename=package://kortex_description/arms/gen3/meshes/HalfArm1_Link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; visual mesh filename=package://kortex_description/arms/gen3/meshes/HalfArm1_Link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
- added link half_arm_2_link, mass 1.1636; collision mesh filename=package://kortex_description/arms/gen3/meshes/HalfArm2_Link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; visual mesh filename=package://kortex_description/arms/gen3/meshes/HalfArm2_Link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
- added link kinova_root
- added link shoulder_link, mass 1.3773; collision mesh filename=package://kortex_description/arms/gen3/meshes/Shoulder_Link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; visual mesh filename=package://kortex_description/arms/gen3/meshes/Shoulder_Link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
- added link spherical_wrist_1_link, mass 0.6781; collision mesh filename=package://kortex_description/arms/gen3/meshes/SphericalWris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; visual mesh filename=package://kortex_description/arms/gen3/meshes/SphericalWris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
- added link spherical_wrist_2_link, mass 0.6781; collision mesh filename=package://kortex_description/arms/gen3/meshes/SphericalWris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; visual mesh filename=package://kortex_description/arms/gen3/meshes/SphericalWris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
Joints:
- added joint FTSensor: type fixed, parent end_effector_link, child ft_sensor_link, origin xyz=0 0 0 rpy=0 0 3.14159265359
- added joint kinova_root_joint: type fixed, parent kinova_root, child base_link
- joint Actuator1: child Shoulder_Link -> shoulder_link
- joint Actuator2: child HalfArm1_Link -> half_arm_1_link; parent Shoulder_Link -> shoulder_link
- joint Actuator3: child HalfArm2_Link -> half_arm_2_link; parent HalfArm1_Link -> half_arm_1_link
- joint Actuator4: child ForeArm_Link -> forearm_link; parent HalfArm2_Link -> half_arm_2_link
- joint Actuator5: child SphericalWrist1_Link -> spherical_wrist_1_link; parent ForeArm_Link -> forearm_link
- joint Actuator6: child SphericalWrist2_Link -> spherical_wrist_2_link; parent SphericalWrist1_Link -> spherical_wrist_1_link
- joint Actuator7: child Bracelet_Link -> bracelet_link; parent SphericalWrist2_Link -> spherical_wrist_2_link
- joint EndEffector: child EndEffector_Link -> end_effector_link; parent Bracelet_Link -> bracelet_link
